File: 100_keyboard.kicad_pcb (KiCad board)
At the start: 2 copper layers, 72.3 x 41.7 mm, 35 parts, among them J1 Conn_01x03, J2 Conn_01x03, J3 USB_B_Micro, J4 Conn_01x05, SW1 SW_Push, U1 mp2359, U2 USBLC6-2SC6, U3 STM32F103RBTx, Y1 16MHz

Commit message: Debug board v0.4 done
Signed-off-by: localcc <work@zloserver.com>
Parts:
- added ?: , test_lib:gh5, F.Cu at (203.1, 42.9)
Connections:
- J3 pad 4: GND -> Net-(J3-Pad4)
Routing:
- net GND: track 49.9 -> 53.4 mm
- added copper zone on F.Cu, net GND
Other:
- board text added: "(C) localcc & zlovantuzu"
- board text added: "Debug Board v0.4"
- board text added: "https://github.com/localcc https://github.com/zlovantuzu"
